File: ov5640_adapter.kicad_pcb (KiCad board)
At the start: 2 copper layers, 30 x 43 mm, 6 parts, among them J1 Conn_02x09_Odd_Even, J2 1-84953-5

Commit message: Added Production files
Other:
- board text added: "OV5640_ADAPTER"
- board text added: "V0.1"
